Commit message: 41515

File: lrmate200id_macro.xacro (robot description, xacro)
@@ -3,20 +3,5 @@
   <xacro:include filename="$(find fanuc_resources)/urdf/common_materials.xacro"/>
   <xacro:macro name="fanuc_lrmate200id" params="prefix">
-    <!-- links: main serial chain -->
-    <link name="${prefix}base_link">
-      <visual>
-        <origin xyz="0 0 0" rpy="0 0 0"/>
-        <geometry>
-          <mesh filename="package://fanuc_lrmate200id_support/meshes/lrmate200id/visual/base_link.stl"/>
-        </geometry>
-        <xacro:material_fanuc_gray28 />
-      </visual>
-      <collision>
-        <origin xyz="0 0 0" rpy="0 0 0"/>
-        <geometry>
-          <mesh filename="package://fanuc_lrmate200id_support/meshes/lrmate200id/collision/base_link.stl"/>
-        </geometry>
-      </collision>
-    </link>
+  <!--###########################################LINK###################################-->
     <link name="${prefix}link_1">
       <visual>
@@ -33,4 +18,9 @@
         </geometry>
       </collision>
+      <inertial>
+            <origin rpy="0 0 0" xyz="0 0 0" />
+            <mass value="2.0" />
+            <inertia ixx="0.01" ixy="0.0" ixz="0.0" iyy="0.01" iyz="0.0" izz="0.01" />
+        </inertial>
     </link>
     <link name="${prefix}link_2">
@@ -48,4 +38,9 @@
         </geometry>
       </collision>
+      <inertial>
+            <origin rpy="0 0 0" xyz="0 0 0" />
+            <mass value="1.5" />
+            <inertia ixx="0.008" ixy="0.0" ixz="0.0" iyy="0.008" iyz="0.0" izz="0.008" />
+        </inertial>
     </link>
     <link name="${prefix}link_3">
@@ -63,4 +58,9 @@
         </geometry>
       </collision>
+      <inertial>
+            <origin rpy="0 0 0" xyz="0 0 0" />
+            <mass value="1.0" />
+            <inertia ixx="0.005" ixy="0.0" ixz="0.0" iyy="0.005" iyz="0.0" izz="0.005" />
+        </inertial>
     </link>
     <link name="${prefix}link_4">
@@ -78,4 +78,9 @@
         </geometry>
       </collision>
+      <inertial>
+            <origin rpy="0 0 0" xyz="0 0 0" />
+            <mass value="1.2" />
+            <inertia ixx="0.007" ixy="0.0" ixz="0.0" iyy="0.007" iyz="0.0" izz="0.007" />
+        </inertial>
     </link>
     <link name="${prefix}link_5">
@@ -93,4 +98,9 @@
         </geometry>
       </collision>
+      <inertial>
+            <origin rpy="0 0 0" xyz="0 0 0" />
+            <mass value="0.8" />
+            <inertia ixx="0.003" ixy="0.0" ixz="0.0" iyy="0.003" iyz="0.0" izz="0.003" />
+        </inertial>
     </link>
     <link name="${prefix}link_6">
@@ -108,6 +118,11 @@
         </geometry>
       </collision>
-    </link>
-	<link name="panda_hand">
+      <inertial>
+            <origin rpy="0 0 0" xyz="0 0 0" />
+            <mass value="0.5" />
+            <inertia ixx="0.002" ixy="0.0" ixz="0.0" iyy="0.002" iyz="0.0" izz="0.002" />
+        </inertial>
+    </link>
+	<link name="gripper_link">
     <visual>
       <geometry>
@@ -120,6 +135,11 @@
       </geometry>
     </collision>
+    <inertial>
+            <origin rpy="0 0 0" xyz="0 0 0" />
+            <mass value="0.3" />
+            <inertia ixx="0.001" ixy="0.0" ixz="0.0" iyy="0.001" iyz="0.0" izz="0.001" />
+        </inertial>
   </link>
-  <link name="panda_leftfinger">
+  <link name="leftfinger">
     <visual>
       <geometry>
@@ -132,6 +152,12 @@
       </geometry>
     </collision>
+    <inertial>
+    <origin xyz="0 0 0" rpy="0 0 0"/>
+            <mass value="0.1" />
+            <origin xyz="0 0 0" rpy="0 0 0" />
+            <inertia ixx="0.03" iyy="0.03" izz="0.03" ixy="0.0" ixz="0.0" iyz="0.0" />
+    </inertial>
   </link>
-  <link name="panda_rightfinger">
+  <link name="rightfinger">
     <visual>
       <origin rpy="0 0 3.141592653589793" xyz="0 0 0"/>
@@ -146,12 +172,19 @@
       </geometry>
     </collision>
+    <inertial>
+    <origin xyz="0 0 0" rpy="0 0 0"/>
+    <mass value="0.1" />
+            <origin xyz="0 0 0" rpy="0 0 0" />
+            <inertia ixx="0.03" iyy="0.03" izz="0.03" ixy="0.0" ixz="0.0" iyz="0.0" />
+ </inertial>
   </link>
-    <!-- joints: main serial chain -->
+    <!--#######################################JOINT#######################################-->
     <joint name="${prefix}joint_1" type="revolute">
       <origin xyz="0 0 0.330" rpy="0 0 0" />
-      <parent link="${prefix}base_link" />
+      <parent link="base_link" />
       <child link="${prefix}link_1" />
       <axis xyz="0 0 1" />
       <limit effort="0" lower="${radians(-170)}" upper="${radians(170)}" velocity="${radians(450)}" />
+    <dynamics damping="20" friction="0.1"/>
     </joint>
     <joint name="${prefix}joint_2" type="revolute">
@@ -161,4 +194,5 @@
       <axis xyz="0 1 0" />
       <limit effort="0" lower="${radians(-100)}" upper="${radians(145)}" velocity="${radians(380)}" />
+    <dynamics damping="20" friction="0.1"/>
     </joint>
     <joint name="${prefix}joint_3" type="revolute">
@@ -168,4 +202,5 @@
       <axis xyz="0 -1 0" />
       <limit effort="0" lower="${radians(-70)}" upper="${radians(205)}" velocity="${radians(520)}" />
+    <dynamics damping="20" friction="0.1"/>
     </joint>
     <joint name="${prefix}joint_4" type="revolute">
@@ -175,4 +210,5 @@
       <axis xyz="-1 0 0"/>
       <limit effort="0" lower="${radians(-190)}" upper="${radians(190)}" velocity="${radians(550)}" />
+    <dynamics damping="20" friction="0.1"/>
     </joint>
     <joint name="${prefix}joint_5" type="revolute">
@@ -182,4 +218,5 @@
       <axis xyz="0 -1 0"/>
       <limit effort="0" lower="${radians(-125)}" upper="${radians(125)}" velocity="${radians(545)}" />
+    <dynamics damping="20" friction="0.1"/>
     </joint>
     <joint name="${prefix}joint_6" type="revolute">
@@ -189,40 +226,176 @@
       <axis xyz="-1 0 0"/>
       <limit effort="0" lower="${radians(-360)}" upper="${radians(360)}" velocity="${radians(1000)}" />
-    </joint>
-    <!-- ROS-Industrial 'base' frame: base_link to Fanuc World Coordinates transform -->
-    <link name="${prefix}base" />
-    <joint name="${prefix}base_link-base" type="fixed">
-      <origin xyz="0 0 0.330" rpy="0 0 0"/>
-      <parent link="${prefix}base_link"/>
-      <child link="${prefix}base"/>
-    </joint>
-    <!-- ROS-Industrial 'flange' frame: attachment point for EEF models -->
+    <dynamics damping="20" friction="0.1"/>
+    </joint>
     <link name="${prefix}flange" />
-    <joint name="${prefix}link_6-flange" type="fixed">
+    <joint name="${prefix}link_6_flange" type="fixed">
       <origin xyz="0 0 0" rpy="0 0 0" />
       <parent link="${prefix}link_6" />
       <child link="${prefix}flange" />
-    </joint>
-    <!-- ROS-Industrial 'tool0' frame: all-zeros tool frame -->
-    <joint name="${prefix}flange-tool0" type="fixed">
+      <dynamics damping="20" friction="0.1"/>
+    </joint>
+    <joint name="${prefix}flange_gripper" type="fixed">
       <origin xyz="0 0 0" rpy="${pi} ${-pi/2.0} 0" />
       <parent link="${prefix}flange" />
-      <child link="panda_hand" />
-    </joint>
-    <joint name="tool0_finger_1" type="prismatic">
-    <parent link="panda_hand"/>
-    <child link="panda_leftfinger"/>
+      <child link="gripper_link" />
+    <dynamics damping="20" friction="0.1"/>
+    </joint>
+    <joint name="finger_joint_1" type="prismatic">
+    <parent link="gripper_link"/>
+    <child link="leftfinger"/>
     <origin rpy="0 0 0" xyz="0 0 0.0584"/>
     <axis xyz="0 1 0"/>
     <limit effort="20" lower="0.0" upper="0.04" velocity="0.2"/>
+    <dynamics damping="20" friction="0.1"/>
   </joint>
-  <joint name="tool0_finger_2" type="prismatic">
-    <parent link="panda_hand"/>
-    <child link="panda_rightfinger"/>
+  <joint name="finger_joint_2" type="prismatic">
+    <parent link="gripper_link"/>
+    <child link="rightfinger"/>
     <origin rpy="0 0 0" xyz="0 0 0.0584"/>
     <axis xyz="0 -1 0"/>
     <limit effort="20" lower="0.0" upper="0.04" velocity="0.2"/>
-    <mimic joint="tool0_finger_1"/>
+    <mimic joint="finger_joint_1"/>
+    <dynamics damping="20" friction="0.1"/>
   </joint>
+  <!--##########################################TRANS####################################-->
+  <transmission name="${prefix}joint_1_trans">
+        <provideFeedback>true</provideFeedback>
+        <implicitSpringDamper>0</implicitSpringDamper>
+        <motorTorqueConstant>0.418</motorTorqueConstant>
+        <type>transmission_interface/SimpleTransmission</type>
+        <joint name="${prefix}joint_1">
+          <hardwareInterface>hardware_interface/PositionJointInterface</hardwareInterface>
+        </joint>
+        <actuator name="${prefix}joint_1_motor">
+          <hardwareInterface>hardware_interface/PositionJointInterface</hardwareInterface>
+          <mechanicalReduction>1</mechanicalReduction>
+        </actuator>
+      </transmission>
+      <transmission name="${prefix}joint_2_trans">
+        <provideFeedback>true</provideFeedback>
+        <implicitSpringDamper>0</implicitSpringDamper>
+        <motorTorqueConstant>0.418</motorTorqueConstant>
+        <type>transmission_interface/SimpleTransmission</type>
+        <joint name="${prefix}joint_2">
+          <hardwareInterface>hardware_interface/PositionJointInterface</hardwareInterface>
+        </joint>
+        <actuator name="${prefix}joint_2_motor">
+          <hardwareInterface>hardware_interface/PositionJointInterface</hardwareInterface>
+          <mechanicalReduction>1</mechanicalReduction>
+        </actuator>
+      </transmission>
+      <transmission name="${prefix}joint_3_trans">
+        <provideFeedback>true</provideFeedback>
+        <implicitSpringDamper>0</implicitSpringDamper>
+        <motorTorqueConstant>0.418</motorTorqueConstant>
+        <type>transmission_interface/SimpleTransmission</type>
+        <joint name="${prefix}joint_3">
+          <hardwareInterface>hardware_interface/PositionJointInterface</hardwareInterface>
+        </joint>
+        <actuator name="${prefix}joint_3_motor">
+          <hardwareInterface>hardware_interface/PositionJointInterface</hardwareInterface>
+          <mechanicalReduction>1</mechanicalReduction>
+        </actuator>
+      </transmission>
+      <transmission name="${prefix}joint_4_trans">
+        <provideFeedback>true</provideFeedback>
+        <implicitSpringDamper>0</implicitSpringDamper>
+        <motorTorqueConstant>0.418</motorTorqueConstant>
+        <type>transmission_interface/SimpleTransmission</type>
+        <joint name="${prefix}joint_4">
+          <hardwareInterface>hardware_interface/PositionJointInterface</hardwareInterface>
+        </joint>
+        <actuator name="${prefix}joint_4_motor">
+          <hardwareInterface>hardware_interface/PositionJointInterface</hardwareInterface>
+          <mechanicalReduction>1</mechanicalReduction>
+        </actuator>
+      </transmission>
+      <transmission name="${prefix}joint_5_trans">
+        <provideFeedback>true</provideFeedback>
+        <implicitSpringDamper>0</implicitSpringDamper>
+        <motorTorqueConstant>0.418</motorTorqueConstant>
+        <type>transmission_interface/SimpleTransmission</type>
+        <joint name="${prefix}joint_5">
+          <hardwareInterface>hardware_interface/PositionJointInterface</hardwareInterface>
+        </joint>
+        <actuator name="${prefix}joint_5_motor">
+          <hardwareInterface>hardware_interface/PositionJointInterface</hardwareInterface>
+          <mechanicalReduction>1</mechanicalReduction>
+        </actuator>
+      </transmission>
+      <transmission name="${prefix}joint_6_trans">
+        <provideFeedback>true</provideFeedback>
+        <implicitSpringDamper>0</implicitSpringDamper>
+        <motorTorqueConstant>0.418</motorTorqueConstant>
+        <type>transmission_interface/SimpleTransmission</type>
+        <joint name="${prefix}joint_6">
+          <hardwareInterface>hardware_interface/PositionJointInterface</hardwareInterface>
+        </joint>
+        <actuator name="${prefix}joint_6_motor">
+          <hardwareInterface>hardware_interface/PositionJointInterface</hardwareInterface>
+          <mechanicalReduction>1</mechanicalReduction>
+        </actuator>
+      </transmission>
+      <transmission name="trans_finger_joint_1">
+        <type>transmission_interface/SimpleTransmission</type>
+        <joint name="finger_joint_1">
+            <hardwareInterface>hardware_interface/PositionJointInterface</hardwareInterface>
+        </joint>
+        <actuator name="finger_joint_1_motor">
+            <hardwareInterface>hardware_interface/PositionJointInterface</hardwareInterface>
+            <mechanicalReduction>1</mechanicalReduction>
+        </actuator>
+    </transmission>
+    <transmission name="trans_finger_joint_2">
+        <type>transmission_interface/SimpleTransmission</type>
+        <joint name="finger_joint_2">
+            <hardwareInterface>hardware_interface/PositionJointInterface</hardwareInterface>
+        </joint>
+        <actuator name="finger_joint_2_motor">
+            <hardwareInterface>hardware_interface/PositionJointInterface</hardwareInterface>
+            <mechanicalReduction>1</mechanicalReduction>
+        </actuator>
+    </transmission>
+  <!--####################################GAZEBO_COLOR##########################################-->
+      <gazebo reference="base_link">
+        <material>Gazebo/Black</material>
+        <selfCollide>true</selfCollide>
+      </gazebo>
+      <gazebo reference="${prefix}link_1">
+        <material>Gazebo/Yellow</material>
+        <selfCollide>true</selfCollide>
+      </gazebo>
+      <gazebo reference="${prefix}link_2">
+        <material>Gazebo/Yellow</material>
+        <selfCollide>true</selfCollide>
+      </gazebo>
+      <gazebo reference="${prefix}link_3">
+        <material>Gazebo/Yellow</material>
+        <selfCollide>true</selfCollide>
+      </gazebo>
+      <gazebo reference="${prefix}link_4">
+        <material>Gazebo/Yellow</material>
+        <selfCollide>true</selfCollide>
+      </gazebo>
+      <gazebo reference="${prefix}link_5">
+        <material>Gazebo/Yellow</material>
+        <selfCollide>true</selfCollide>
+      </gazebo>
+      <gazebo reference="${prefix}link_6">
+        <material>Gazebo/Yellow</material>
+        <selfCollide>true</selfCollide>
+      </gazebo>
+      <gazebo reference="gripper_link">
+        <material>Gazebo/Black</material>
+        <selfCollide>true</selfCollide>
+      </gazebo>
+      <gazebo reference="leftfinger">
+        <material>Gazebo/Black</material>
+        <selfCollide>true</selfCollide>
+      </gazebo>
+      <gazebo reference="rightfinger">
+        <material>Gazebo/Black</material>
+        <selfCollide>true</selfCollide>
+      </gazebo>
   </xacro:macro>
 </robot>

File: test/lrmate200id.xacro (robot description, xacro)
@@ -5,5 +5,5 @@
        xmlns:xacro="http://ros.org/wiki/xacro">
   <xacro:arg name="robot_namespace" default="" />
-  <xacro:include filename="$(find fanuc_lrmate200id_support)/urdf/lrmate200id_macro.xacro"/>
+  <xacro:include filename="$(find fanuc_lrmate200id_support)/urdf/test/lrmate200id_macro.xacro"/>
   <!--##############################################################################-->
   <link name="base_link">

File: test_URDF/lrmate200id_macro.xacro (robot description, xacro)
@@ -124,5 +124,5 @@
         </inertial>
     </link>
-	<link name="gripper_link">
+	<link name="panda_hand">
     <visual>
       <geometry>
@@ -141,5 +141,5 @@
         </inertial>
   </link>
-  <link name="leftfinger">
+  <link name="panda_leftfinger">
     <visual>
       <geometry>
@@ -159,5 +159,5 @@
     </inertial>
   </link>
-  <link name="rightfinger">
+  <link name="panda_rightfinger">
     <visual>
       <origin rpy="0 0 3.141592653589793" xyz="0 0 0"/>
@@ -228,13 +228,20 @@
     <dynamics damping="20" friction="0.1"/>
     </joint>
-    <joint name="${prefix}link_6_gripper_link" type="fixed">
+    <link name="${prefix}flange" />
+    <joint name="${prefix}link_6-flange" type="fixed">
+      <origin xyz="0 0 0" rpy="0 0 0" />
+      <parent link="${prefix}link_6" />
+      <child link="${prefix}flange" />
+      <dynamics damping="20" friction="0.1"/>
+    </joint>
+    <joint name="${prefix}link6-tool0" type="fixed">
       <origin xyz="0 0 0" rpy="${pi} ${-pi/2.0} 0" />
-      <parent link="${prefix}link_6" />
-      <child link="gripper_link" />
-    <dynamics damping="20" friction="0.1"/>
-    </joint>
-    <joint name="finger_joint_1" type="prismatic">
-    <parent link="gripper_link"/>
-    <child link="leftfinger"/>
+      <parent link="${prefix}flange" />
+      <child link="panda_hand" />
+    <dynamics damping="20" friction="0.1"/>
+    </joint>
+    <joint name="tool0_finger_1" type="prismatic">
+    <parent link="panda_hand"/>
+    <child link="panda_leftfinger"/>
     <origin rpy="0 0 0" xyz="0 0 0.0584"/>
     <axis xyz="0 1 0"/>
@@ -242,11 +249,11 @@
     <dynamics damping="20" friction="0.1"/>
   </joint>
-  <joint name="finger_joint_2" type="prismatic">
-    <parent link="gripper_link"/>
-    <child link="rightfinger"/>
+  <joint name="tool0_finger_2" type="prismatic">
+    <parent link="panda_hand"/>
+    <child link="panda_rightfinger"/>
     <origin rpy="0 0 0" xyz="0 0 0.0584"/>
     <axis xyz="0 -1 0"/>
     <limit effort="20" lower="0.0" upper="0.04" velocity="0.2"/>
-    <mimic joint="finger_joint_1"/>
+    <!-- <mimic joint="tool0_finger_1"/> -->
     <dynamics damping="20" friction="0.1"/>
   </joint>
@@ -330,20 +337,20 @@
         </actuator>
       </transmission>
-      <transmission name="trans_finger_joint_1">
-        <type>transmission_interface/SimpleTransmission</type>
-        <joint name="finger_joint_1">
+      <transmission name="trans_tool0_finger_1">
+        <type>transmission_interface/SimpleTransmission</type>
+        <joint name="tool0_finger_1">
             <hardwareInterface>hardware_interface/PositionJointInterface</hardwareInterface>
         </joint>
-        <actuator name="finger_joint_1_motor">
+        <actuator name="tool0_finger_1_motor">
             <hardwareInterface>hardware_interface/PositionJointInterface</hardwareInterface>
             <mechanicalReduction>1</mechanicalReduction>
         </actuator>
     </transmission>
-    <transmission name="trans_finger_joint_2">
-        <type>transmission_interface/SimpleTransmission</type>
-        <joint name="finger_joint_2">
+    <transmission name="trans_tool0_finger_2">
+        <type>transmission_interface/SimpleTransmission</type>
+        <joint name="tool0_finger_2">
             <hardwareInterface>hardware_interface/PositionJointInterface</hardwareInterface>
         </joint>
-        <actuator name="finger_joint_2_motor">
+        <actuator name="tool0_finger_2_motor">
             <hardwareInterface>hardware_interface/PositionJointInterface</hardwareInterface>
             <mechanicalReduction>1</mechanicalReduction>
@@ -379,13 +386,13 @@
         <selfCollide>true</selfCollide>
       </gazebo>
-      <gazebo reference="gripper_link">
+      <gazebo reference="panda_hand">
         <material>Gazebo/Black</material>
         <selfCollide>true</selfCollide>
       </gazebo>
-      <gazebo reference="leftfinger">
+      <gazebo reference="panda_leftfinger">
         <material>Gazebo/Black</material>
         <selfCollide>true</selfCollide>
       </gazebo>
-      <gazebo reference="rightfinger">
+      <gazebo reference="panda_rightfinger">
         <material>Gazebo/Black</material>
         <selfCollide>true</selfCollide>
